Commit message: Added robotiq. It can appear in RVIZ but can't in Gazebo.

File: src/robotiq/robotiq_2f_85_gripper_visualization/urdf/robotiq_arg2f.xacro (robot description, xacro)
@@ -3,9 +3,18 @@
   <xacro:macro name="robotiq_arg2f_base_link" params="prefix">
     <link name="${prefix}robotiq_arg2f_base_link">
-      <inertial>
+     <inertial>
         <origin xyz="8.625E-08 -4.6583E-06 0.03145" rpy="0 0 0" />
         <mass value="0.22652" />
-        <inertia ixx="0.00020005" ixy="-4.2442E-10" ixz="-2.9069E-10" iyy="0.00017832" iyz="-3.4402E-08" izz="0.00013478" />
+        <inertia ixx="0.00020005" ixy="-4.2442E-10" ixz="-2.9069E-10"
+                 iyx="0.00000" iyy="0.00017832" iyz="-3.4402E-08"
+                 izx="0.00000" izy="0.00000" izz="0.00013478" />
       </inertial>
+<!--      <inertial>
+        <mass value="0.636951" />
+        <origin xyz="0.0 0.0 0.0" />
+        <inertia ixx = "0.000380" ixy = "0.000000" ixz = "0.000000"
+                 iyx = "0.000000" iyy = "0.001110" iyz = "0.000000"
+                 izx = "0.000000" izy = "0.000000" izz = "0.001171" />
+      </inertial>   -->
       <visual>
         <origin xyz="0 0 0" rpy="0 0 0" />

File: src/robotiq/robotiq_2f_85_gripper_visualization/urdf/robotiq_arg2f_85_model_macro.xacro (robot description, xacro)
@@ -2,11 +2,15 @@
 <robot xmlns:xacro="http://ros.org/wiki/xacro">
   <xacro:include filename="$(find robotiq_2f_85_gripper_visualization)/urdf/robotiq_arg2f_transmission.xacro" />
+<!-- definition of robotiq_arg2f_85_gazebo (add)-->
+  <xacro:include filename="$(find robotiq_2f_85_gripper_visualization)/urdf/robotiq_arg2f_85.gazebo.xacro" />
   <xacro:macro name="outer_knuckle" params="prefix fingerprefix stroke">
     <link name="${prefix}${fingerprefix}_outer_knuckle">
-      <!--<inertial>
+      <inertial>
         <origin xyz="-0.000200000000003065 0.0199435877845359 0.0292245259211331" rpy="0 0 0" />
         <mass value="0.00853198276973456" />
-        <inertia ixx="2.89328108496468E-06" ixy="-1.57935047237397E-19" ixz="-1.93980378593255E-19" iyy="1.86719750325683E-06" iyz="-1.21858577871576E-06" izz="1.21905238907251E-06" />
-        </inertial> -->
+        <inertia ixx="2.89328108496468E-06" ixy="-1.57935047237397E-19" ixz="-1.93980378593255E-19"
+                 iyx="0.00000" iyy="1.86719750325683E-06" iyz="-1.21858577871576E-06"
+                 izx="0.00000" izy="0.00000" izz="1.21905238907251E-06" />
+      </inertial>
       <visual>
         <origin xyz="0 0 0" rpy="0 0 0" />
@@ -28,9 +32,11 @@
   <xacro:macro name="outer_finger" params="prefix fingerprefix stroke">
     <link name="${prefix}${fingerprefix}_outer_finger">
-      <!--<inertial>
+      <inertial>
         <origin xyz="0.00030115855001899 0.0373907951953854 -0.0208027427000385" rpy="0 0 0" />
         <mass value="0.022614240507152" />
-        <inertia ixx="1.52518312458174E-05" ixy="9.76583423954399E-10" ixz="-5.43838577022588E-10" iyy="6.17694243867776E-06" iyz="6.78636130740228E-06" izz="1.16494917907219E-05" />
-        </inertial> -->
+        <inertia ixx="1.52518312458174E-05" ixy="9.76583423954399E-10" ixz="-5.43838577022588E-10"
+                 iyx="0.00000" iyy="6.17694243867776E-06" iyz="6.78636130740228E-06"
+                 izx="0.00000" izy="0.00000" izz="1.16494917907219E-05" />
+      </inertial>
       <visual>
         <origin xyz="0 0 0" rpy="0 0 0" />
@@ -52,9 +58,11 @@
   <xacro:macro name="inner_knuckle" params="prefix fingerprefix stroke">
     <link name="${prefix}${fingerprefix}_inner_knuckle">
-      <!--<inertial>
+      <inertial>
         <origin xyz="0.000123011831763771 0.0507850843201817 0.00103968640075166" rpy="0 0 0" />
        <mass value="0.0271177346495152" />
-        <inertia ixx="2.61910379223783E-05" ixy="-2.43616858946494E-07" ixz="-6.37789906117123E-09" iyy="2.8270243746167E-06" iyz="-5.37200748039765E-07" izz="2.83695868220296E-05" />
-        </inertial> -->
+        <inertia ixx="2.61910379223783E-05" ixy="-2.43616858946494E-07" ixz="-6.37789906117123E-09"
+                 iyx="0.00000" iyy="2.8270243746167E-06" iyz="-5.37200748039765E-07"
+                 izx="0.00000" izy="0.00000" izz="2.83695868220296E-05" />
+      </inertial>
       <visual>
         <origin xyz="0 0 0" rpy="0 0 0" />
@@ -76,9 +84,11 @@
   <xacro:macro name="inner_finger" params="prefix fingerprefix stroke">
     <link name="${prefix}${fingerprefix}_inner_finger">
-      <!--<inertial>
+      <inertial>
         <origin xyz="0.000299999999999317 0.0160078233491243 -0.0136945669206257" rpy="0 0 0" />
         <mass value="0.0104003125914103" />
-        <inertia ixx="2.71909453810972E-06" ixy="1.35402465472579E-21" ixz="-7.1817349065269E-22" iyy="7.69100314106116E-07" iyz="6.74715432769696E-07" izz="2.30315190420171E-06" />
-        </inertial> -->
+        <inertia ixx="2.71909453810972E-06" ixy="1.35402465472579E-21" ixz="-7.1817349065269E-22"
+                 iyx="0.00000" iyy="7.69100314106116E-07" iyz="6.74715432769696E-07"
+                 izx="0.00000" izy="0.00000" izz="2.30315190420171E-06" />
+      </inertial>
       <visual>
         <origin xyz="0 0 0" rpy="0 0 0" />
@@ -101,5 +111,12 @@
   <xacro:macro name="inner_finger_pad" params="prefix fingerprefix">
     <link name="${prefix}${fingerprefix}_inner_finger_pad">
-      <visual>
+     <inertial>
+       <mass value="0.018491" />
+       <origin xyz="0.0 0.0 0.0" />
+       <inertia ixx = "0.000009" ixy = "-0.000001" ixz = "0.000000"
+                iyy = "0.000001" iyz = "0.000000"
+                izz = "0.000010" />
+     </inertial>
+     <visual>
         <origin xyz="0 0 0" rpy="0 0 0" />
         <geometry>
@@ -188,4 +205,23 @@
     <xacro:right_outer_knuckle_joint prefix="${prefix}"/>
     <xacro:robotiq_arg2f_transmission prefix="${prefix}"/>
-  </xacro:macro>
+<!-- definition of robotiq_arg2f_85_gazebo (add)-->
+    <xacro:robotiq_arg2f_85_gazebo prefix="${prefix}" />
+  </xacro:macro>
+<!--
+  <gazebo>
+    <plugin name="gazebo_grasp_fix" filename="libgazebo_grasp_fix.so">
+        <arm>
+          <arm_name>gripper_arm</arm_name>
+          <palm_link>ee_link</palm_link>
+          <gripper_link>right_inner_finger_pad</gripper_link>
+          <gripper_link>left_inner_finger_pad</gripper_link>
+        </armt>
+      <forces_angle_tolerance>100</forces_angle_tolerance>
+      <update_rate>2</update_rate>
+      <max_grip_count>2</max_grip_count>
+      <release_tolerance>0.005</release_tolerance>
+      <disable_collisions_on_attach>true</disable_collisions_on_attach>
+      <contact_topic>__default_topic__</contact_topic>
+    </plugin>
+  </gazebo> -->
 </robot>

File: src/robotiq/robotiq_2f_85_gripper_visualization/urdf/robotiq_arg2f_transmission.xacro (robot description, xacro)
@@ -5,5 +5,5 @@
       <type>transmission_interface/SimpleTransmission</type>
       <joint name="${prefix}finger_joint">
-        <hardwareInterface>PositionJointInterface</hardwareInterface>
+        <hardwareInterface>hardware_interface/PositionJointInterface</hardwareInterface>
       </joint>
       <actuator name="${prefix}finger_joint_motor">

File: src/universal_robot/ur_description/urdf/ur5_joint_limited_robot.urdf.xacro (robot description, xacro)
@@ -7,4 +7,7 @@
   <!-- ur5 -->
   <xacro:include filename="$(find ur_description)/urdf/ur5.urdf.xacro" />
+  <!-- robotiq_2f_85 (add) -->
+  <xacro:include filename="$(find robotiq_2f_85_gripper_visualization)/urdf/robotiq_arg2f_85_model.xacro" />
+<!--  <param name="robot_description" command="$(find xacro)/xacro $(find robotiq_2f_85_gripper_visualization)/urdf/robotiq_arg2f_85_model.xacro" />  -->
   <!-- arm -->
   <xacro:ur5_robot prefix="" joint_limited="true"
@@ -23,3 +26,9 @@
     <origin xyz="0.0 0.0 0.0" rpy="0.0 0.0 0.0" />
   </joint>
+  <!-- robotiq_2f_85 (add) -->
+  <joint name="base_link_joint" type="fixed">
+    <parent link="ee_link" />
+    <child link = "robotiq_arg2f_base_link" />
+    <origin xyz="0.01 0 0" rpy="0 ${pi/2} 0"/>
+  </joint>
 </robot>
