Commit message: improve collapse : remove mimic and disable coupler_link collision

File: src/robotiq/robotiq_2f_model/model/robotiq_2f_85.urdf.xacro (robot description, xacro)
@@ -62,4 +62,5 @@
 		</link>
                 <gazebo reference="${name}_base">
+                    <selfCollide>true</selfCollide>
                     <implicitSpringDamper>1</implicitSpringDamper>
                     <mu1>100000</mu1>
@@ -106,4 +107,5 @@
 		</link>
                 <gazebo reference="${name}_right_driver">
+                    <selfCollide>true</selfCollide>
                     <implicitSpringDamper>1</implicitSpringDamper>
                     <mu1>100000</mu1>
@@ -150,12 +152,13 @@
 			</xacro:unless>
 			<xacro:if value="${precise_collision}">
-				<collision>
+<!--				<collision>
 					<geometry>
 						<mesh filename="package://robotiq_2f_model/model/meshes/2f85/collision/coupler.stl" scale="0.001 0.001 0.001"/>
 					</geometry>
-				</collision>
+				</collision> -->
 			</xacro:if>
 		</link>
                 <gazebo reference="${name}_right_coupler">
+                    <selfCollide>true</selfCollide>
                     <implicitSpringDamper>1</implicitSpringDamper>
                     <mu1>100000</mu1>
@@ -171,7 +174,7 @@
 			<axis xyz="1 0 0"/>
 			<limit lower="${-170 * 3.141592 / 180}" upper="${170 * 3.141592 / 180}" effort="1000" velocity="${110 * 3.141592 / 180}" />
-			<xacro:unless value="${adaptive_transmission}">
+<!--			<xacro:unless value="${adaptive_transmission}">
 			<mimic joint="${name}_right_driver_joint" multiplier="-1"/>
-			</xacro:unless>
+			</xacro:unless> -->
 		</joint>
 		<link name="${name}_right_follower">
@@ -209,4 +212,5 @@
 		</link>
                 <gazebo reference="${name}_right_follower">
+                    <selfCollide>true</selfCollide>
                     <implicitSpringDamper>1</implicitSpringDamper>
                     <mu1>100000</mu1>
@@ -253,8 +257,9 @@
 			</link>
                 	<gazebo reference="${name}_right_pad">
-                  	  <implicitSpringDamper>1</implicitSpringDamper>
-                 	   <mu1>100000</mu1>
+                            <selfCollide>true</selfCollide>
+                  	    <implicitSpringDamper>1</implicitSpringDamper>
+                 	    <mu1>100000</mu1>
                 	    <mu2>100000</mu2>
-                 	   <kp>100000000.0</kp>
+                 	    <kp>100000000.0</kp>
                 	    <kd>1.0</kd>
              		</gazebo>
@@ -266,7 +271,7 @@
 			<axis xyz="1 0 0"/>
 			<limit lower="${-170 * 3.141592 / 180}" upper="${170 * 3.141592 / 180}" effort="1000" velocity="${110 * 3.141592 / 180}" />
-			<xacro:unless value="${adaptive_transmission}">
+<!--			<xacro:unless value="${adaptive_transmission}">
 			<mimic joint="${name}_right_driver_joint" multiplier="1"/>
-			</xacro:unless>
+			</xacro:unless> -->
 		</joint>
 		<link name="${name}_right_spring_link">
@@ -300,4 +305,5 @@
 		</link>
                 <gazebo reference="${name}_right_spring_link">
+                    <selfCollide>true</selfCollide>
                     <implicitSpringDamper>1</implicitSpringDamper>
                     <mu1>100000</mu1>
@@ -313,7 +319,7 @@
 			<axis xyz="1 0 0"/>
 			<limit lower="${0 * 3.141592 / 180}" upper="${50 * 3.141592 / 180}" effort="1000" velocity="${110 * 3.141592 / 180}" />
-			<xacro:unless value="${adaptive_transmission}">
+<!--			<xacro:unless value="${adaptive_transmission}">
 			<mimic joint="${name}_right_driver_joint" multiplier="1"/>
-			</xacro:unless>
+			</xacro:unless> -->
 		</joint>
 		<link name="${name}_left_driver">
@@ -347,4 +353,5 @@
 		</link>
                 <gazebo reference="${name}_left_driver">
+                    <selfCollide>true</selfCollide>
                     <implicitSpringDamper>1</implicitSpringDamper>
                     <mu1>100000</mu1>
@@ -390,13 +397,14 @@
 			</xacro:unless>
 			<xacro:if value="${precise_collision}">
-				<collision>
+<!--				<collision>
 				<origin xyz="0 0.0 0.025" rpy="-1.7 0 0"/>
 					<geometry>
 						<mesh filename="package://robotiq_2f_model/model/meshes/2f85/collision/coupler.stl" scale="0.001 0.001 0.001"/>
 					</geometry>
-				</collision>
+				</collision> -->
 			</xacro:if>
 		</link>
                 <gazebo reference="${name}_left_coupler">
+                    <selfCollide>true</selfCollide>
                     <implicitSpringDamper>1</implicitSpringDamper>
                     <mu1>100000</mu1>
@@ -413,7 +421,7 @@
 			<axis xyz="1 0 0"/>
 			<limit lower="${-170 * 3.141592 / 180}" upper="${170 * 3.141592 / 180}" effort="1000" velocity="${110 * 3.141592 / 180}" />
-			<xacro:unless value="${adaptive_transmission}">
+<!--			<xacro:unless value="${adaptive_transmission}">
 			<mimic joint="${name}_right_driver_joint" multiplier="-1"/>
-			</xacro:unless>
+			</xacro:unless> -->
 		</joint>
 		<link name="${name}_left_follower">
@@ -451,4 +459,5 @@
 		</link>
                 <gazebo reference="${name}_left_follower">
+                    <selfCollide>true</selfCollide>
                     <implicitSpringDamper>1</implicitSpringDamper>
                     <mu1>100000</mu1>
@@ -495,4 +504,5 @@
 			</link>
                 	<gazebo reference="${name}_left_pad">
+                                <selfCollide>true</selfCollide>
                    	        <implicitSpringDamper>1</implicitSpringDamper>
                   	        <mu1>100000</mu1>
@@ -508,7 +518,7 @@
 			<axis xyz="1 0 0"/>
 			<limit lower="${-170 * 3.141592 / 180}" upper="${170 * 3.141592 / 180}" effort="17600" velocity="${110 * 3.141592 / 180}" />
-			<xacro:unless value="${adaptive_transmission}">
+<!--			<xacro:unless value="${adaptive_transmission}">
 			<mimic joint="${name}_right_driver_joint" multiplier="1"/>
-			</xacro:unless>
+			</xacro:unless> -->
 		</joint>
 		<link name="${name}_left_spring_link">
@@ -542,4 +552,5 @@
 		</link>
                 <gazebo reference="${name}_left_spring_link">
+                        <selfCollide>true</selfCollide>
                    	<implicitSpringDamper>1</implicitSpringDamper>
                   	<mu1>100000</mu1>
@@ -555,4 +566,54 @@
 				</joint>
 				<actuator name="${name}_right_driver_motor">
+					<mechanicalReduction>1</mechanicalReduction>
+					<hardwareInterface>PositionJointInterface</hardwareInterface>
+				</actuator>
+			</transmission>
+			<transmission name="${name}_left_driver_trans">
+				<type>transmission_interface/SimpleTransmission</type>
+				<joint name="${name}_left_driver_joint">
+					<hardwareInterface>hardware_interface/PositionJointInterface</hardwareInterface>
+				</joint>
+				<actuator name="${name}_left_driver_motor">
+					<mechanicalReduction>1</mechanicalReduction>
+					<hardwareInterface>PositionJointInterface</hardwareInterface>
+				</actuator>
+			</transmission>
+			<transmission name="${name}_right_follower_trans">
+				<type>transmission_interface/SimpleTransmission</type>
+				<joint name="${name}_right_follower_joint">
+					<hardwareInterface>hardware_interface/PositionJointInterface</hardwareInterface>
+				</joint>
+				<actuator name="${name}_right_follower_motor">
+					<mechanicalReduction>1</mechanicalReduction>
+					<hardwareInterface>PositionJointInterface</hardwareInterface>
+				</actuator>
+			</transmission>
+			<transmission name="${name}_left_follower_trans">
+				<type>transmission_interface/SimpleTransmission</type>
+				<joint name="${name}_left_follower_joint">
+					<hardwareInterface>hardware_interface/PositionJointInterface</hardwareInterface>
+				</joint>
+				<actuator name="${name}_left_follower_motor">
+					<mechanicalReduction>1</mechanicalReduction>
+					<hardwareInterface>PositionJointInterface</hardwareInterface>
+				</actuator>
+			</transmission>
+			<transmission name="${name}_right_spring_link_trans">
+				<type>transmission_interface/SimpleTransmission</type>
+				<joint name="${name}_right_spring_link_joint">
+					<hardwareInterface>hardware_interface/PositionJointInterface</hardwareInterface>
+				</joint>
+				<actuator name="${name}_right_spring_link_motor">
+					<mechanicalReduction>1</mechanicalReduction>
+					<hardwareInterface>PositionJointInterface</hardwareInterface>
+				</actuator>
+			</transmission>
+			<transmission name="${name}_left_spring_link_trans">
+				<type>transmission_interface/SimpleTransmission</type>
+				<joint name="${name}_left_spring_link_joint">
+					<hardwareInterface>hardware_interface/PositionJointInterface</hardwareInterface>
+				</joint>
+				<actuator name="${name}_left_spring_link_motor">
 					<mechanicalReduction>1</mechanicalReduction>
 					<hardwareInterface>PositionJointInterface</hardwareInterface>
@@ -605,5 +666,5 @@
 					<mimicJoint>add_left_joint</mimicJoint>
 					<multiplier>-1</multiplier>
-				</plugin> -->
+				</plugin>
 				<plugin name="${name}_right_follower_joint_plugin" filename="libroboticsgroup_gazebo_mimic_joint_plugin.so">
 					<joint>${name}_right_driver_joint</joint>
@@ -632,5 +693,5 @@
 					<mimicJoint>${name}_left_driver_joint</mimicJoint>
 					<multiplier>1</multiplier>
-				</plugin>
+				</plugin> -->
                                  <!-- add for pegasus closed plugin
 				<plugin name="${name}_right_ClosedLoopPlugin" filename="libpegasus_gazebo_closed_loop_plugin.so">

Commit message: add the small door model and open by position control and gazebo grasp plugin

File: src/robotiq/robotiq_2f_model/model/robotiq_2f_85.urdf.xacro (robot description, xacro)
@@ -127,5 +127,5 @@
 			<child link="${name}_right_coupler"/>
 			<axis xyz="1 0 0"/>
-			<limit lower="${-170 * 3.141592 / 180}" upper="${170 * 3.141592 / 180}" effort="17600" velocity="${110 * 3.141592 / 180}" />
+			<limit lower="${-170 * 3.141592 / 180}" upper="${170 * 3.141592 / 180}" effort="1000" velocity="${110 * 3.141592 / 180}" />
 		</joint>
 		</xacro:if>
@@ -216,6 +216,10 @@
                     <mu1>100000</mu1>
                     <mu2>100000</mu2>
-                    <kp>100000000.0</kp>
+                    <kp>1.0</kp>
                     <kd>1.0</kd>
+<!--                    <mu1>100000</mu1>
+               	        <mu2>100000</mu2>
+               	        <kp>100000000.0</kp>
+               	        <kd>1.0</kd> -->
                 </gazebo>
 		<xacro:if value="${with_pads}">
@@ -261,6 +265,10 @@
                  	    <mu1>100000</mu1>
                 	    <mu2>100000</mu2>
-                 	    <kp>100000000.0</kp>
-                	    <kd>1.0</kd>
+               	            <kp>1.0</kp>
+                  	    <kd>1.0</kd>
+<!--                 	    <mu1>100000</mu1>
+                	    <mu2>100000</mu2>
+                  	        <kp>100000000.0</kp>
+                  	        <kd>1.0</kd> -->
              		</gazebo>
 		</xacro:if>
@@ -373,5 +381,5 @@
 			<child link="${name}_left_coupler"/>
 			<axis xyz="1 0 0"/>
-			<limit lower="${-170 * 3.141592 / 180}" upper="${170 * 3.141592 / 180}" effort="17600" velocity="${110 * 3.141592 / 180}" />
+			<limit lower="${-170 * 3.141592 / 180}" upper="${170 * 3.141592 / 180}" effort="1000" velocity="${110 * 3.141592 / 180}" />
 		</joint>
 		</xacro:if>
@@ -463,6 +471,10 @@
                     <mu1>100000</mu1>
                     <mu2>100000</mu2>
-                    <kp>100000000.0</kp>
+                    <kp>1.0</kp>
                     <kd>1.0</kd>
+<!--                    <mu1>100000</mu1>
+               	        <mu2>100000</mu2>
+               	        <kp>100000000.0</kp>
+               	        <kd>1.0</kd> -->
                 </gazebo>
 		<xacro:if value="${with_pads}">
@@ -508,6 +520,10 @@
                   	        <mu1>100000</mu1>
                   	        <mu2>100000</mu2>
+                  	        <kp>1.0</kp>
+                  	        <kd>1.0</kd>
+<!--                  	        <mu1>100000</mu1>
+                  	        <mu2>100000</mu2>
                   	        <kp>100000000.0</kp>
-                  	        <kd>1.0</kd>
+                  	        <kd>1.0</kd> -->
              		</gazebo>
 		</xacro:if>
@@ -517,5 +533,5 @@
 			<child link="${name}_left_spring_link"/>
 			<axis xyz="1 0 0"/>
-			<limit lower="${-170 * 3.141592 / 180}" upper="${170 * 3.141592 / 180}" effort="17600" velocity="${110 * 3.141592 / 180}" />
+			<limit lower="${-170 * 3.141592 / 180}" upper="${170 * 3.141592 / 180}" effort="1000" velocity="${110 * 3.141592 / 180}" />
 <!--			<xacro:unless value="${adaptive_transmission}">
 			<mimic joint="${name}_right_driver_joint" multiplier="1"/>
@@ -563,9 +579,11 @@
 				<type>transmission_interface/SimpleTransmission</type>
 				<joint name="${name}_right_driver_joint">
-					<hardwareInterface>hardware_interface/PositionJointInterface</hardwareInterface>
+					<hardwareInterface>hardware_interface/EffortJointInterface</hardwareInterface>
+<!--					<hardwareInterface>hardware_interface/PositionJointInterface</hardwareInterface> -->
 				</joint>
 				<actuator name="${name}_right_driver_motor">
 					<mechanicalReduction>1</mechanicalReduction>
-					<hardwareInterface>PositionJointInterface</hardwareInterface>
+					<hardwareInterface>EffortJointInterface</hardwareInterface>
+<!--					<hardwareInterface>PositionJointInterface</hardwareInterface> -->
 				</actuator>
 			</transmission>
@@ -573,9 +591,11 @@
 				<type>transmission_interface/SimpleTransmission</type>
 				<joint name="${name}_left_driver_joint">
-					<hardwareInterface>hardware_interface/PositionJointInterface</hardwareInterface>
+					<hardwareInterface>hardware_interface/EffortJointInterface</hardwareInterface>
+<!--					<hardwareInterface>hardware_interface/PositionJointInterface</hardwareInterface> -->
 				</joint>
 				<actuator name="${name}_left_driver_motor">
 					<mechanicalReduction>1</mechanicalReduction>
-					<hardwareInterface>PositionJointInterface</hardwareInterface>
+					<hardwareInterface>EffortJointInterface</hardwareInterface>
+<!--					<hardwareInterface>PositionJointInterface</hardwareInterface> -->
 				</actuator>
 			</transmission>
@@ -583,9 +603,11 @@
 				<type>transmission_interface/SimpleTransmission</type>
 				<joint name="${name}_right_follower_joint">
-					<hardwareInterface>hardware_interface/PositionJointInterface</hardwareInterface>
+					<hardwareInterface>hardware_interface/EffortJointInterface</hardwareInterface>
+<!--					<hardwareInterface>hardware_interface/PositionJointInterface</hardwareInterface> -->
 				</joint>
 				<actuator name="${name}_right_follower_motor">
 					<mechanicalReduction>1</mechanicalReduction>
-					<hardwareInterface>PositionJointInterface</hardwareInterface>
+					<hardwareInterface>EffortJointInterface</hardwareInterface>
+<!--					<hardwareInterface>PositionJointInterface</hardwareInterface> -->
 				</actuator>
 			</transmission>
@@ -593,9 +615,11 @@
 				<type>transmission_interface/SimpleTransmission</type>
 				<joint name="${name}_left_follower_joint">
-					<hardwareInterface>hardware_interface/PositionJointInterface</hardwareInterface>
+					<hardwareInterface>hardware_interface/EffortJointInterface</hardwareInterface>
+<!--					<hardwareInterface>hardware_interface/PositionJointInterface</hardwareInterface> -->
 				</joint>
 				<actuator name="${name}_left_follower_motor">
 					<mechanicalReduction>1</mechanicalReduction>
-					<hardwareInterface>PositionJointInterface</hardwareInterface>
+					<hardwareInterface>EffortJointInterface</hardwareInterface>
+<!--					<hardwareInterface>PositionJointInterface</hardwareInterface> -->
 				</actuator>
 			</transmission>
@@ -603,9 +627,11 @@
 				<type>transmission_interface/SimpleTransmission</type>
 				<joint name="${name}_right_spring_link_joint">
-					<hardwareInterface>hardware_interface/PositionJointInterface</hardwareInterface>
+					<hardwareInterface>hardware_interface/EffortJointInterface</hardwareInterface>
+<!--					<hardwareInterface>hardware_interface/PositionJointInterface</hardwareInterface> -->
 				</joint>
 				<actuator name="${name}_right_spring_link_motor">
 					<mechanicalReduction>1</mechanicalReduction>
-					<hardwareInterface>PositionJointInterface</hardwareInterface>
+					<hardwareInterface>EffortJointInterface</hardwareInterface>
+<!--					<hardwareInterface>PositionJointInterface</hardwareInterface> -->
 				</actuator>
 			</transmission>
@@ -613,9 +639,11 @@
 				<type>transmission_interface/SimpleTransmission</type>
 				<joint name="${name}_left_spring_link_joint">
-					<hardwareInterface>hardware_interface/PositionJointInterface</hardwareInterface>
+					<hardwareInterface>hardware_interface/EffortJointInterface</hardwareInterface>
+<!--					<hardwareInterface>hardware_interface/PositionJointInterface</hardwareInterface> -->
 				</joint>
 				<actuator name="${name}_left_spring_link_motor">
 					<mechanicalReduction>1</mechanicalReduction>
-					<hardwareInterface>PositionJointInterface</hardwareInterface>
+					<hardwareInterface>EffortJointInterface</hardwareInterface>
+<!--					<hardwareInterface>PositionJointInterface</hardwareInterface> -->
 				</actuator>
 			</transmission>
@@ -709,4 +737,19 @@
                                         <rotation>0.00 -0.00 0.00</rotation>
 				</plugin> -->
+   	                        <plugin name="gazebo_grasp_fix" filename="libgazebo_grasp_fix.so">
+                                  <arm>
+                                        <arm_name>gripper_arm</arm_name>
+                                        <palm_link>${parent}</palm_link>
+                                        <gripper_link>${name}_right_follower</gripper_link>
+                                        <gripper_link>${name}_left_follower</gripper_link>
+                                  </arm>
+	                          <forces_angle_tolerance>100</forces_angle_tolerance>
+	                          <update_rate>2</update_rate>
+	                          <grip_count_threshold>1</grip_count_threshold>
+	                          <max_grip_count>2</max_grip_count>
+	                          <release_tolerance>0.005</release_tolerance>
+	                          <disable_collisions_on_attach>true</disable_collisions_on_attach>
+	                          <contact_topic>__default_topic__</contact_topic>
+	                        </plugin>
 			</gazebo>
 		</xacro:unless>
