Commit message: add open ai ros

File: src/robotiq/robotiq_2f_model/model/robotiq_2f_85.urdf.xacro (robot description, xacro)
@@ -579,10 +579,10 @@
 				<type>transmission_interface/SimpleTransmission</type>
 				<joint name="${name}_right_driver_joint">
-					<hardwareInterface>hardware_interface/EffortJointInterface</hardwareInterface>
+					<hardwareInterface>hardware_interface/PositionJointInterface</hardwareInterface>
 <!--					<hardwareInterface>hardware_interface/PositionJointInterface</hardwareInterface> -->
 				</joint>
 				<actuator name="${name}_right_driver_motor">
 					<mechanicalReduction>1</mechanicalReduction>
-					<hardwareInterface>EffortJointInterface</hardwareInterface>
+					<hardwareInterface>PositionJointInterface</hardwareInterface>
 <!--					<hardwareInterface>PositionJointInterface</hardwareInterface> -->
 				</actuator>
@@ -591,10 +591,10 @@
 				<type>transmission_interface/SimpleTransmission</type>
 				<joint name="${name}_left_driver_joint">
-					<hardwareInterface>hardware_interface/EffortJointInterface</hardwareInterface>
+					<hardwareInterface>hardware_interface/PositionJointInterface</hardwareInterface>
 <!--					<hardwareInterface>hardware_interface/PositionJointInterface</hardwareInterface> -->
 				</joint>
 				<actuator name="${name}_left_driver_motor">
 					<mechanicalReduction>1</mechanicalReduction>
-					<hardwareInterface>EffortJointInterface</hardwareInterface>
+					<hardwareInterface>PositionJointInterface</hardwareInterface>
 <!--					<hardwareInterface>PositionJointInterface</hardwareInterface> -->
 				</actuator>
@@ -603,10 +603,10 @@
 				<type>transmission_interface/SimpleTransmission</type>
 				<joint name="${name}_right_follower_joint">
-					<hardwareInterface>hardware_interface/EffortJointInterface</hardwareInterface>
+					<hardwareInterface>hardware_interface/PositionJointInterface</hardwareInterface>
 <!--					<hardwareInterface>hardware_interface/PositionJointInterface</hardwareInterface> -->
 				</joint>
 				<actuator name="${name}_right_follower_motor">
 					<mechanicalReduction>1</mechanicalReduction>
-					<hardwareInterface>EffortJointInterface</hardwareInterface>
+					<hardwareInterface>PositionJointInterface</hardwareInterface>
 <!--					<hardwareInterface>PositionJointInterface</hardwareInterface> -->
 				</actuator>
@@ -615,10 +615,10 @@
 				<type>transmission_interface/SimpleTransmission</type>
 				<joint name="${name}_left_follower_joint">
-					<hardwareInterface>hardware_interface/EffortJointInterface</hardwareInterface>
+					<hardwareInterface>hardware_interface/PositionJointInterface</hardwareInterface>
 <!--					<hardwareInterface>hardware_interface/PositionJointInterface</hardwareInterface> -->
 				</joint>
 				<actuator name="${name}_left_follower_motor">
 					<mechanicalReduction>1</mechanicalReduction>
-					<hardwareInterface>EffortJointInterface</hardwareInterface>
+					<hardwareInterface>PositionJointInterface</hardwareInterface>
 <!--					<hardwareInterface>PositionJointInterface</hardwareInterface> -->
 				</actuator>
@@ -627,10 +627,10 @@
 				<type>transmission_interface/SimpleTransmission</type>
 				<joint name="${name}_right_spring_link_joint">
-					<hardwareInterface>hardware_interface/EffortJointInterface</hardwareInterface>
+					<hardwareInterface>hardware_interface/PositionJointInterface</hardwareInterface>
 <!--					<hardwareInterface>hardware_interface/PositionJointInterface</hardwareInterface> -->
 				</joint>
 				<actuator name="${name}_right_spring_link_motor">
 					<mechanicalReduction>1</mechanicalReduction>
-					<hardwareInterface>EffortJointInterface</hardwareInterface>
+					<hardwareInterface>PositionJointInterface</hardwareInterface>
 <!--					<hardwareInterface>PositionJointInterface</hardwareInterface> -->
 				</actuator>
@@ -639,10 +639,10 @@
 				<type>transmission_interface/SimpleTransmission</type>
 				<joint name="${name}_left_spring_link_joint">
-					<hardwareInterface>hardware_interface/EffortJointInterface</hardwareInterface>
+					<hardwareInterface>hardware_interface/PositionJointInterface</hardwareInterface>
 <!--					<hardwareInterface>hardware_interface/PositionJointInterface</hardwareInterface> -->
 				</joint>
 				<actuator name="${name}_left_spring_link_motor">
 					<mechanicalReduction>1</mechanicalReduction>
-					<hardwareInterface>EffortJointInterface</hardwareInterface>
+					<hardwareInterface>PositionJointInterface</hardwareInterface>
 <!--					<hardwareInterface>PositionJointInterface</hardwareInterface> -->
 				</actuator>

File: src/universal_robot/ur_description/urdf/ur5.urdf.xacro (robot description, xacro)
@@ -286,5 +286,6 @@
       <axis xyz="0 1 0" />
       <xacro:unless value="${joint_limited}">
-        <limit lower="${-2.0 * pi}" upper="${2.0 * pi}" effort="28.0" velocity="3.2"/>
+        <limit lower="${-2.0 * pi}" upper="${2.0 * pi}" effort="0.001" velocity="3.2"/>
+<!--        <limit lower="${-2.0 * pi}" upper="${2.0 * pi}" effort="28.0" velocity="3.2"/> -->
         <xacro:if value="${safety_limits}">
           <safety_controller soft_lower_limit="${-2.0 * pi + safety_pos_margin}" soft_upper_limit="${2.0 * pi - safety_pos_margin}" k_position="${safety_k_position}" k_velocity="0.0"/>

Commit message: implement openairos to door opening task

File: src/robotiq/robotiq_2f_model/model/robotiq_2f_85.urdf.xacro (robot description, xacro)
@@ -39,5 +39,5 @@
 				</geometry>
 			</visual>
-			<xacro:unless value="${precise_collision}">
+<!--			<xacro:unless value="${precise_collision}">
 			<collision>
 				<origin xyz="0 0 0.015" rpy="0 0 0"/>
@@ -59,5 +59,5 @@
 				</geometry>
 			</collision>
-			</xacro:if>
+			</xacro:if> -->
 		</link>
                 <gazebo reference="${name}_base">
@@ -90,5 +90,5 @@
 				</geometry>
 			</visual>
-			<xacro:unless value="${precise_collision}">
+<!--			<xacro:unless value="${precise_collision}">
 			<collision>
 				<origin xyz="0 0.01 0" rpy="-0.1 0 0"/>
@@ -104,5 +104,5 @@
 				</geometry>
 			</collision>
-			</xacro:if>
+			</xacro:if> -->
 		</link>
                 <gazebo reference="${name}_right_driver">
@@ -196,5 +196,4 @@
 			<collision>
 				<origin xyz="0 0 0" />
-<!--				<origin xyz="0 -0.01 0.022" rpy="0 0 0"/> -->
 				<geometry>
 					<box size="0.002 0.0015 0.0048"/>
@@ -296,5 +295,5 @@
 				</geometry>
 			</visual>
-			<xacro:unless value="${precise_collision}">
+<!--			<xacro:unless value="${precise_collision}">
 			<collision>
 				<origin xyz="0 0.025 0.015" rpy="-0.7068 0 0"/>
@@ -310,5 +309,5 @@
 				</geometry>
 			</collision>
-			</xacro:if>
+			</xacro:if> -->
 		</link>
                 <gazebo reference="${name}_right_spring_link">
@@ -344,5 +343,5 @@
 				</geometry>
 			</visual>
-			<xacro:unless value="${precise_collision}">
+<!--			<xacro:unless value="${precise_collision}">
 			<collision>
 				<origin xyz="0 0.01 0" rpy="-0.1 0 0"/>
@@ -358,5 +357,5 @@
 				</geometry>
 			</collision>
-			</xacro:if>
+			</xacro:if>  -->
 		</link>
                 <gazebo reference="${name}_left_driver">
@@ -551,5 +550,5 @@
 				</geometry>
 			</visual>
-			<xacro:unless value="${precise_collision}">
+<!--			<xacro:unless value="${precise_collision}">
 			<collision>
 				<origin xyz="0 0.025 0.015" rpy="-0.7068 0 0"/>
@@ -565,5 +564,5 @@
 				</geometry>
 			</collision>
-			</xacro:if>
+			</xacro:if>  -->
 		</link>
                 <gazebo reference="${name}_left_spring_link">
@@ -745,10 +744,12 @@
                                   </arm>
 	                          <forces_angle_tolerance>100</forces_angle_tolerance>
-	                          <update_rate>2</update_rate>
-	                          <grip_count_threshold>1</grip_count_threshold>
-	                          <max_grip_count>2</max_grip_count>
+	                          <update_rate>0.01</update_rate>
+<!-- /pos_traj_controller/command = 100Hz, /gazebo/model_states & /gazebo/link_states = 1kHz, /joint_states = 50Hz -->
+	                          <grip_count_threshold>0.01</grip_count_threshold>
+	                          <max_grip_count>1</max_grip_count>
 	                          <release_tolerance>0.005</release_tolerance>
 	                          <disable_collisions_on_attach>true</disable_collisions_on_attach>
-	                          <contact_topic>__default_topic__</contact_topic>
+	                          <contact_topic>grasp_plugin</contact_topic>
+<!---	                          <contact_topic>__default_topic__</contact_topic> -->
 	                        </plugin>
 			</gazebo>

File: src/universal_robot/ur_description/urdf/ur5.urdf.xacro (robot description, xacro)
@@ -86,9 +86,9 @@
         </material>
       </visual>
-      <collision>
+<!--      <collision>
         <geometry>
           <mesh filename="package://ur_description/meshes/ur5/collision/base.stl" />
         </geometry>
-      </collision>
+      </collision>  -->
       <xacro:c_inertia radius="0.06" length="0.05" mass="${base_mass}">
         <origin xyz="0.0 0.0 0.0" rpy="0 0 0" />
@@ -123,9 +123,9 @@
         </material>
       </visual>
-      <collision>
+<!--      <collision>
         <geometry>
           <mesh filename="package://ur_description/meshes/ur5/collision/shoulder.stl" />
         </geometry>
-      </collision>
+      </collision>  -->
       <xacro:c_inertia radius="0.06" length="0.15" mass="${shoulder_mass}">
         <origin xyz="0.0 0.0 0.0" rpy="0 0 0" />
@@ -160,9 +160,9 @@
         </material>
       </visual>
-      <collision>
+<!--      <collision>
         <geometry>
           <mesh filename="package://ur_description/meshes/ur5/collision/upperarm.stl" />
         </geometry>
-      </collision>
+      </collision>  -->
       <xacro:c_inertia radius="0.06" length="0.56" mass="${upper_arm_mass}">
         <origin xyz="0.0 0.0 0.28" rpy="0 0 0" />
@@ -197,9 +197,9 @@
         </material>
       </visual>
-      <collision>
+<!--      <collision>
         <geometry>
           <mesh filename="package://ur_description/meshes/ur5/collision/forearm.stl" />
         </geometry>
-      </collision>
+      </collision>  -->
       <xacro:c_inertia radius="0.06" length="${-a3}" mass="${forearm_mass}">
         <origin xyz="0.0 0.0 ${-a3/2}" rpy="0 0 0" />
@@ -234,9 +234,9 @@
         </material>
       </visual>
-      <collision>
+<!--      <collision>
         <geometry>
           <mesh filename="package://ur_description/meshes/ur5/collision/wrist1.stl" />
         </geometry>
-      </collision>
+      </collision> -->
       <xacro:c_inertia radius="0.06" length="0.12" mass="${wrist_1_mass}">
         <origin xyz="0.0 ${wrist_1_length} 0.0" rpy="0 0 0" />
@@ -271,9 +271,9 @@
         </material>
       </visual>
-      <collision>
+<!--      <collision>
         <geometry>
           <mesh filename="package://ur_description/meshes/ur5/collision/wrist2.stl" />
         </geometry>
-      </collision>
+      </collision> -->
       <xacro:c_inertia radius="0.06" length="0.12" mass="${wrist_2_mass}">
         <origin xyz="0.0 0.0 ${wrist_2_length}" rpy="0 0 0" />
@@ -286,5 +286,5 @@
       <axis xyz="0 1 0" />
       <xacro:unless value="${joint_limited}">
-        <limit lower="${-2.0 * pi}" upper="${2.0 * pi}" effort="0.001" velocity="3.2"/>
+        <limit lower="${-2.0 * pi}" upper="${2.0 * pi}" effort="28.0" velocity="3.2"/>
 <!--        <limit lower="${-2.0 * pi}" upper="${2.0 * pi}" effort="28.0" velocity="3.2"/> -->
         <xacro:if value="${safety_limits}">
@@ -309,9 +309,9 @@
         </material>
       </visual>
-      <collision>
+<!--      <collision>
         <geometry>
           <mesh filename="package://ur_description/meshes/ur5/collision/wrist3.stl" />
         </geometry>
-      </collision>
+      </collision> -->
       <xacro:c_inertia radius="0.0375" length="0.0345" mass="${wrist_3_mass}">
         <origin xyz="0.0 ${wrist_3_length - 0.0345/2} 0.0" rpy="${pi/2} 0 0" />
@@ -323,4 +323,15 @@
       <origin xyz="0.0 ${wrist_3_length} 0.0" rpy="0.0 0.0 ${pi/2.0}" />
     </joint>
+    <gazebo reference="${prefix}wrist_3_joint">
+        <provideFeedback>true</provideFeedback>
+    </gazebo>
+    <!-- The ft_sensor plugin -->
+    <gazebo>
+        <plugin name="ft_sensor" filename="libgazebo_ros_ft_sensor.so">
+            <updateRate>0</updateRate>	<!-- updateRate must be 0 for avoiding stop when reset the simulation -->
+            <topicName>ft_sensor_topic</topicName>
+            <jointName>wrist_3_joint</jointName>
+        </plugin>
+    </gazebo>
     <link name="${prefix}ee_link">
       <collision>

File: src/universal_robot/ur_description/urdf/ur5_joint_limited_robot.urdf.xacro (robot description, xacro)
@@ -11,4 +11,14 @@
   <!-- arm -->
   <xacro:ur5_robot prefix="" joint_limited="true"
+    shoulder_pan_lower_limit="${-0.2}" shoulder_pan_upper_limit="${1.8}"
+    shoulder_lift_lower_limit="${-2.7}" shoulder_lift_upper_limit="${0.2}"
+    elbow_joint_lower_limit="${-0.2}" elbow_joint_upper_limit="${2.7}"
+    wrist_1_lower_limit="${-0.7}" wrist_1_upper_limit="${0.3}"
+    wrist_2_lower_limit="${-0.2}" wrist_2_upper_limit="${2.2}"
+    wrist_3_lower_limit="${-1.8}" wrist_3_upper_limit="${1.5}"
+    transmission_hw_interface="$(arg transmission_hw_interface)"
+  />
+  <!-- arm
+  <xacro:ur5_robot prefix="" joint_limited="true"
     shoulder_pan_lower_limit="${-pi}" shoulder_pan_upper_limit="${pi}"
     shoulder_lift_lower_limit="${-pi}" shoulder_lift_upper_limit="${pi}"
@@ -18,5 +28,5 @@
     wrist_3_lower_limit="${-pi}" wrist_3_upper_limit="${pi}"
     transmission_hw_interface="$(arg transmission_hw_interface)"
-  />
+  /> -->
   <link name="world" />
   <joint name="world_joint" type="fixed">
