Commit message: confirmed that robotiq could operate

File: src/robotiq/robotiq_2f_robot/robot/simple_rq2f85.urdf.xacro (robot description, xacro)
@@ -7,5 +7,5 @@
 	<xacro:robotiq_2f_85 name="simple_gripper" parent="wrist_3_link" precise_collision="true" adaptive_transmission="false">
 <!--  0.0823 = wrist_3_length = d6 -->
-                <origin xyz="0 0.0823 0" rpy="${pi/-2.0} 0 0"/>
+                <origin xyz="0 0.0823 0" rpy="${pi/-2.0} ${pi/2.0} 0"/>
 	</xacro:robotiq_2f_85>
 </robot>

Commit message: 20210224 update

File: src/robotiq/robotiq_2f_robot/robot/simple_rq2f85.urdf.xacro (robot description, xacro)
@@ -6,6 +6,8 @@
 		<origin xyz="0 0 0" rpy="0 0 0"/>  -->
 	<xacro:robotiq_2f_85 name="simple_gripper" parent="wrist_3_link" precise_collision="true" adaptive_transmission="false">
-<!--  0.0823 = wrist_3_length = d6 -->
-                <origin xyz="0 0.0823 0" rpy="${pi/-2.0} ${pi/2.0} 0"/>
+<!--  0.037 = FT300_length -->
+<!--  0.0823 + 0.037 = 0.1193 -->
+                <origin xyz="0 0.1193 0" rpy="${pi/-2.0} ${pi/2.0} 0"/>
+<!--                <origin xyz="0 0.0823 0" rpy="${pi/-2.0} ${pi/2.0} 0"/> -->
 	</xacro:robotiq_2f_85>
 </robot>

File: src/universal_robot/ur_description/urdf/ur5.urdf.xacro (robot description, xacro)
@@ -86,9 +86,9 @@
         </material>
       </visual>
-      <collision>
+<!--      <collision>
         <geometry>
           <mesh filename="package://ur_description/meshes/ur5/collision/base.stl" />
         </geometry>
-      </collision>
+      </collision> -->
       <xacro:c_inertia radius="0.06" length="0.05" mass="${base_mass}">
         <origin xyz="0.0 0.0 0.0" rpy="0 0 0" />
@@ -123,9 +123,9 @@
         </material>
       </visual>
-      <collision>
+<!--      <collision>
         <geometry>
           <mesh filename="package://ur_description/meshes/ur5/collision/shoulder.stl" />
         </geometry>
-      </collision>
+      </collision> -->
       <xacro:c_inertia radius="0.06" length="0.15" mass="${shoulder_mass}">
         <origin xyz="0.0 0.0 0.0" rpy="0 0 0" />
@@ -160,9 +160,9 @@
         </material>
       </visual>
-      <collision>
+<!--     <collision>
         <geometry>
           <mesh filename="package://ur_description/meshes/ur5/collision/upperarm.stl" />
         </geometry>
-      </collision>
+      </collision> -->
       <xacro:c_inertia radius="0.06" length="0.56" mass="${upper_arm_mass}">
         <origin xyz="0.0 0.0 0.28" rpy="0 0 0" />
@@ -197,9 +197,9 @@
         </material>
       </visual>
-      <collision>
+<!--      <collision>
         <geometry>
           <mesh filename="package://ur_description/meshes/ur5/collision/forearm.stl" />
         </geometry>
-      </collision>
+      </collision> -->
       <xacro:c_inertia radius="0.06" length="${-a3}" mass="${forearm_mass}">
         <origin xyz="0.0 0.0 ${-a3/2}" rpy="0 0 0" />
@@ -234,9 +234,9 @@
         </material>
       </visual>
-      <collision>
+<!--      <collision>
         <geometry>
           <mesh filename="package://ur_description/meshes/ur5/collision/wrist1.stl" />
         </geometry>
-      </collision>
+      </collision> -->
       <xacro:c_inertia radius="0.06" length="0.12" mass="${wrist_1_mass}">
         <origin xyz="0.0 ${wrist_1_length} 0.0" rpy="0 0 0" />
@@ -271,9 +271,9 @@
         </material>
       </visual>
-      <collision>
+<!--      <collision>
         <geometry>
           <mesh filename="package://ur_description/meshes/ur5/collision/wrist2.stl" />
         </geometry>
-      </collision>
+      </collision> -->
       <xacro:c_inertia radius="0.06" length="0.12" mass="${wrist_2_mass}">
         <origin xyz="0.0 0.0 ${wrist_2_length}" rpy="0 0 0" />
@@ -308,9 +308,9 @@
         </material>
       </visual>
-      <collision>
+<!--      <collision>
         <geometry>
           <mesh filename="package://ur_description/meshes/ur5/collision/wrist3.stl" />
         </geometry>
-      </collision>
+      </collision> -->
       <xacro:c_inertia radius="0.0375" length="0.0345" mass="${wrist_3_mass}">
         <origin xyz="0.0 ${wrist_3_length - 0.0345/2} 0.0" rpy="${pi/2} 0 0" />
@@ -334,10 +334,10 @@
     </gazebo>
     <link name="${prefix}ee_link">
-      <collision>
+<!--      <collision>
         <geometry>
           <box size="0.01 0.01 0.01"/>
         </geometry>
         <origin rpy="0 0 0" xyz="-0.01 0 0"/>
-      </collision>
+      </collision> -->
     </link>
     <xacro:ur_arm_transmission prefix="${prefix}" hw_interface="${transmission_hw_interface}" />
